File: PanelLed/PanelLed.kicad_pcb (KiCad board)
At the start: 2 copper layers, 21.6 x 15.2 mm, 7 parts, among them J1 Conn_01x02_Male, J2 Conn_01x02_Male, J3 Conn_01x02_Male

Commit message: Boards sent to be built.
Changed lines of the file:
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@@
     (solder_mask_min_width 0.25)
     (aux_axis_origin 0 0)
-    (visible_elements FFFFFF7F)
+    (visible_elements 7FFFFFFF)
     (pcbplotparams
       (layerselection 0x010fc_ffffffff)
@@
       (outputformat 1)
       (mirror false)
-      (drillshape 1)
+      (drillshape 0)
       (scaleselection 1)
       (outputdirectory ""))
@@
     (descr "LED, diameter 5.0mm, 2 pins, http://cdn-reichelt.de/documents/datenblatt/A500/LL-504BC2E-009.pdf")
     (tags "LED diameter 5.0mm 2 pins")
-    (fp_text reference D1 (at 1.27 -3.96) (layer F.SilkS)
+    (fp_text reference D1 (at -1.905 2.54) (layer F.SilkS)
       (effects (font (size 1 1) (thickness 0.15)))
     )
@@
     (tags "resistor handsolder")
     (attr smd)
-    (fp_text reference R1 (at 0 1.65 90) (layer B.SilkS)
+    (fp_text reference R1 (at -2.6035 0 180) (layer B.SilkS)
       (effects (font (size 1 1) (thickness 0.15)) (justify mirror))
     )
@@
     (descr "JST EH series connector, B2B-EH-A (http://www.jst-mfg.com/product/pdf/eng/eEH.pdf), generated with kicad-footprint-generator")
     (tags "connector JST EH vertical")
-    (fp_text reference J3 (at 1.25 2.8) (layer B.SilkS)
+    (fp_text reference J3 (at -4.1275 -0.3175) (layer B.SilkS)
       (effects (font (size 1 1) (thickness 0.15)) (justify mirror))
     )
@@
     (descr "JST EH series connector, B2B-EH-A (http://www.jst-mfg.com/product/pdf/eng/eEH.pdf), generated with kicad-footprint-generator")
     (tags "connector JST EH vertical")
-    (fp_text reference J2 (at 1.25 2.8 180) (layer B.SilkS)
+    (fp_text reference J2 (at -1.27 -3.4925 180) (layer B.SilkS)
       (effects (font (size 1 1) (thickness 0.15)) (justify mirror))
     )
@@
     (descr "JST EH series connector, B2B-EH-A (http://www.jst-mfg.com/product/pdf/eng/eEH.pdf), generated with kicad-footprint-generator")
     (tags "connector JST EH vertical")
-    (fp_text reference J1 (at 1.25 2.8) (layer B.SilkS)
-      (effects (font (size 1 1) (thickness 0.15)) (justify mirror))
-    )
+    (fp_text reference J1 (at -1.905 -3.4925) (layer B.SilkS)
+      (effects (font (size 1 1) (thickness 0.15)) (justify mirror))
+    )
