File: PanelSwitch/PanelSwitch.sch (KiCad schematic (older format))
At the start: 16 parts, among them J1 Conn_01x02_Male, J2 Conn_01x02_Male, J3 Conn_01x02_Male

Commit message: Boards sent to be built.
Connections:
- net labels added: A0, A1, A2, A3, B0, B1, B2, B3
Changed lines of the file:
@@
 Wire Wire Line
 	4200 4350 4500 4350
+Text Label 4300 3900 0    50   ~ 0
+A
 Text Label 4300 4350 0    50   ~ 0
+B
+Wire Wire Line
+	3600 3500 3900 3500
+Text Label 3700 3600 0    50   ~ 0
 A
-Text Label 4300 3900 0    50   ~ 0
+Wire Wire Line
+	3600 3600 3900 3600
+Text Label 3700 3500 0    50   ~ 0
 B
 Wire Wire Line
-	3600 3500 3900 3500
-Text Label 3700 3500 0    50   ~ 0
+	3600 3950 3900 3950
+Text Label 3700 4050 0    50   ~ 0
 A
 Wire Wire Line
-	3600 3600 3900 3600
-Text Label 3700 3600 0    50   ~ 0
-B
-Wire Wire Line
-	3600 3950 3900 3950
+	3600 4050 3900 4050
 Text Label 3700 3950 0    50   ~ 0
-A
-Wire Wire Line
-	3600 4050 3900 4050
-Text Label 3700 4050 0    50   ~ 0
 B
 $Comp
@@
 U 1 1 6525498D
 P 7000 3900
-F 0 "R5" V 6950 3750 50  0000 C CNN
+F 0 "R5" V 6900 3900 50  0000 C CNN
 F 1 "10k" V 7000 3900 50  0000 C CNN
 F 2 "Resistor_SMD:R_0805_2012Metric_Pad1.15x1.40mm_HandSolder" V 6930 3900 50  0001 C CNN
@@
 U 1 1 65258B2F
 P 7000 4200
-F 0 "R6" V 6950 4050 50  0000 C CNN
+F 0 "R6" V 6900 4200 50  0000 C CNN
 F 1 "10k" V 7000 4200 50  0000 C CNN
 F 2 "Resistor_SMD:R_0805_2012Metric_Pad1.15x1.40mm_HandSolder" V 6930 4200 50  0001 C CNN
@@
 U 1 1 6525927C
 P 7000 4500
-F 0 "R7" V 6950 4350 50  0000 C CNN
+F 0 "R7" V 6900 4500 50  0000 C CNN
 F 1 "10k" V 7000 4500 50  0000 C CNN
 F 2 "Resistor_SMD:R_0805_2012Metric_Pad1.15x1.40mm_HandSolder" V 6930 4500 50  0001 C CNN
@@
 U 1 1 65259F8B
 P 7000 4800
-F 0 "R8" V 6950 4650 50  0000 C CNN
+F 0 "R8" V 6900 4800 50  0000 C CNN
 F 1 "10k" V 7000 4800 50  0000 C CNN
 F 2 "Resistor_SMD:R_0805_2012Metric_Pad1.15x1.40mm_HandSolder" V 6930 4800 50  0001 C CNN
@@
 Wire Wire Line
 	5100 3950 5550 3950
+Text Label 5100 3750 0    50   ~ 0
+A0
+Text Label 5100 3850 0    50   ~ 0
+A1
+Text Label 5100 3950 0    50   ~ 0
+A2
+Text Label 5100 4050 0    50   ~ 0
+A3
+Text Label 5100 4200 0    50   ~ 0
+B0
+Text Label 5100 4300 0    50   ~ 0
+B1
+Text Label 5100 4400 0    50   ~ 0
+B2
+Text Label 5100 4500 0    50   ~ 0
+B3
 $EndSCHEMATC
