File: Sensor/Thermocouple/Thermocouple.kicad_pcb (KiCad board)
At the start: 2 copper layers, 28.6 x 26 mm, 17 parts, among them J1 Conn_02x04_Odd_Even, J2 Conn_01x02_Female, U1 MIC5225, U2 MAX31856

Commit message: Boards sent to be built.
Parts:
- R1, R2: value R -> 100
Changed lines of the file:
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@@
     (add_net /~Fault)
     (add_net GND)
+    (add_net "Net-(U1-Pad4)")
+    (add_net "Net-(U2-Pad6)")
   )
   (module 0MiscParts:TSSOP-14_4.4x5mm_P0.65mm_MAX (layer F.Cu)
@@
       (effects (font (size 1 1) (thickness 0.15)))
     )
-    (fp_text value R (at 0 1.65) (layer F.Fab)
+    (fp_text value 100 (at 0 1.65) (layer F.Fab)
       (effects (font (size 1 1) (thickness 0.15)))
     )
@@
       (effects (font (size 1 1) (thickness 0.15)))
     )
-    (fp_text value R (at 0 1.65 90) (layer F.Fab)
+    (fp_text value 100 (at 0 1.65 90) (layer F.Fab)
       (effects (font (size 1 1) (thickness 0.15)))
     )
