File: Sensor/Thermocouple/Thermocouple.sch (KiCad schematic (older format))
At the start: 17 parts, among them J1 Conn_02x04_Odd_Even, J2 Conn_01x02_Female, U1 MIC5225, U2 MAX31856

Commit message: Boards sent to be built.
Parts:
- R1, R2: value R -> 100
Changed lines of the file:
@@
 P 7750 4100
 F 0 "R1" V 7543 4100 50  0000 C CNN
-F 1 "R" V 7634 4100 50  0000 C CNN
+F 1 "100" V 7634 4100 50  0000 C CNN
 F 2 "Resistor_SMD:R_0805_2012Metric_Pad1.15x1.40mm_HandSolder" V 7680 4100 50  0001 C CNN
 F 3 "~" H 7750 4100 50  0001 C CNN
@@
 P 7750 4400
 F 0 "R2" V 7543 4400 50  0000 C CNN
-F 1 "R" V 7634 4400 50  0000 C CNN
+F 1 "100" V 7634 4400 50  0000 C CNN
 F 2 "Resistor_SMD:R_0805_2012Metric_Pad1.15x1.40mm_HandSolder" V 7680 4400 50  0001 C CNN
 F 3 "~" H 7750 4400 50  0001 C CNN
