File: OutputMega/OutputMega.sch (KiCad schematic (older format))
At the start: 134 parts, among them J1 Control, J10 Conn_02x13_Top_Bottom, J11 EStop Sig1 JST2H, J12 MegaProMiniR, J13 JTAG, J14 Dbg, J15 EStop Rly JST2H, J16 Sp Rly 1 JST2H, J17 Sp Rly 2 JST2H, J18 Step Disable JST2H, J19 EStop Sig0 JST2H, J2 EStop JST3H, J20 EStop Sig1 JST2H, J21 Conn_01x06_Male, J22 Conn_02x05_Odd_Even, J23 Sw 12v 1 JST2H, J24 Sw 12v 2 JST2H, J25 Pilot JST2H, J26 VFD Dir JST3H, J27 VFD Ctl JST3H, J3 EStop Rst JST2H, J4 TmrTest, J5 DbgPort, J6 RemPort, J7 12VIn, J8 PwrIn, J9 MegaProMiniL, K1 G6S-2, K2 G6S-2, K3 G6S-2, Q1 2N7002, Q10 2N7002, Q11 2N7002, Q12 2N7002, Q13 2N7002, Q2 2N7002, Q3 2N7002, Q4 2N7002, Q5 2N7002, Q6 2N7002, Q7 2N7002, Q8 2N7002, Q9 2N7002, U1 74HCT123, U10 MC34072AP, U2 74LS08, U3 LD1117S50TR_SOT223, U4 74LVC2G00, U5 74AUC2G34, U6 74AUC2G34, U7 74LVC2G157, U8 74LS08, U9 TLV9351

Commit message: Output Mega layout completed.
Parts:
- removed C8: .1uf, Capacitor_SMD:C_0805_2012Metric_Pad1.15x1.40mm_HandSolder, symbol Device:C
- J1: footprint Connector_JST:JST_EH_S5B-EH_1x05_P2.50mm_Horizontal -> 0MiscParts:JST_EH_S5B-EH_1x05_P2.50mm_Horizontal
- J11, J15, J16, J17, J18, J19, J20, J23, J24, J25, J3, J7, J8: footprint Connector_JST:JST_EH_S2B-EH_1x02_P2.50mm_Horizontal -> 0MiscParts:JST_EH_S2B-EH_1x02_P2.50mm_Horizontal
- J2, J26, J27, J6: footprint Connector_JST:JST_EH_S3B-EH_1x03_P2.50mm_Horizontal -> 0MiscParts:JST_EH_S3B-EH_1x03_P2.50mm_Horizontal
- J5: footprint Connector_JST:JST_EH_S4B-EH_1x04_P2.50mm_Horizontal -> 0MiscParts:JST_EH_S4B-EH_1x04_P2.50mm_Horizontal
Connections:
- net labels added: ESRR, ESSR, EStopRlyExt
- net labels removed: EGR, ESR, EStopRlyDrv
Other:
- moved on the sheet: C7, D17, R20
Changed lines of the file:
@@
 F 0 "J6" H 750 3150 50  0000 R CNN
 F 1 "RemPort" H 1100 3150 50  0000 R CNN
-F 2 "Connector_JST:JST_EH_S3B-EH_1x03_P2.50mm_Horizontal" H 800 3400 50  0001 C CNN
+F 2 "0MiscParts:JST_EH_S3B-EH_1x03_P2.50mm_Horizontal" H 800 3400 50  0001 C CNN
 F 3 "~" H 800 3400 50  0001 C CNN
 	1    800  3400
@@
 F 0 "J5" H 650 2350 50  0000 R CNN
 F 1 "DbgPort" H 1000 2350 50  0000 R CNN
-F 2 "Connector_JST:JST_EH_S4B-EH_1x04_P2.50mm_Horizontal" H 800 2700 50  0001 C CNN
+F 2 "0MiscParts:JST_EH_S4B-EH_1x04_P2.50mm_Horizontal" H 800 2700 50  0001 C CNN
 F 3 "~" H 800 2700 50  0001 C CNN
 	1    800  2700
@@
 F 0 "J7" H 2592 1135 50  0000 C CNN
 F 1 "12VIn" H 2600 750 50  0000 C CNN
-F 2 "Connector_JST:JST_EH_S2B-EH_1x02_P2.50mm_Horizontal" H 2700 950 50  0001 C CNN
+F 2 "0MiscParts:JST_EH_S2B-EH_1x02_P2.50mm_Horizontal" H 2700 950 50  0001 C CNN
 F 3 "~" H 2700 950 50  0001 C CNN
 	1    2700 950
@@
 F 0 "J8" H 3692 1085 50  0000 C CNN
 F 1 "PwrIn" H 3700 700 50  0000 C CNN
-F 2 "Connector_JST:JST_EH_S2B-EH_1x02_P2.50mm_Horizontal" H 3800 900 50  0001 C CNN
+F 2 "0MiscParts:JST_EH_S2B-EH_1x02_P2.50mm_Horizontal" H 3800 900 50  0001 C CNN
 F 3 "~" H 3800 900 50  0001 C CNN
 	1    3800 900
@@
 F 0 "J1" H 600 4200 50  0000 C CNN
 F 1 "Control" H 800 4200 50  0000 C CNN
-F 2 "Connector_JST:JST_EH_S5B-EH_1x05_P2.50mm_Horizontal" H 650 4550 50  0001 C CNN
+F 2 "0MiscParts:JST_EH_S5B-EH_1x05_P2.50mm_Horizontal" H 650 4550 50  0001 C CNN
 F 3 "~" H 650 4550 50  0001 C CNN
 	1    650  4550
@@
 F 0 "J2" H 650 6400 50  0000 R CNN
 F 1 "EStop JST3H" H 1150 6400 50  0000 R CNN
-F 2 "Connector_JST:JST_EH_S3B-EH_1x03_P2.50mm_Horizontal" H 700 6650 50  0001 C CNN
+F 2 "0MiscParts:JST_EH_S3B-EH_1x03_P2.50mm_Horizontal" H 700 6650 50  0001 C CNN
 F 3 "~" H 700 6650 50  0001 C CNN
 	1    700  6650
@@
 F 0 "J3" H 650 7600 50  0000 R CNN
 F 1 "EStop Rst JST2H" H 1300 7600 50  0000 R CNN
-F 2 "Connector_JST:JST_EH_S2B-EH_1x02_P2.50mm_Horizontal" H 700 7850 50  0001 C CNN
+F 2 "0MiscParts:JST_EH_S2B-EH_1x02_P2.50mm_Horizontal" H 700 7850 50  0001 C CNN
 F 3 "~" H 700 7850 50  0001 C CNN
 	1    700  7850
@@
 F 0 "J19" H 10200 4800 50  0000 R CNN
 F 1 "EStop Sig0 JST2H" H 10600 4600 50  0000 R CNN
-F 2 "Connector_JST:JST_EH_S2B-EH_1x02_P2.50mm_Horizontal" H 10250 4800 50  0001 C CNN
+F 2 "0MiscParts:JST_EH_S2B-EH_1x02_P2.50mm_Horizontal" H 10250 4800 50  0001 C CNN
 F 3 "~" H 10250 4800 50  0001 C CNN
 	1    10250 4800
@@
 F 0 "J20" H 10200 5200 50  0000 R CNN
 F 1 "EStop Sig1 JST2H" H 10600 5000 50  0000 R CNN
-F 2 "Connector_JST:JST_EH_S2B-EH_1x02_P2.50mm_Horizontal" H 10250 5200 50  0001 C CNN
+F 2 "0MiscParts:JST_EH_S2B-EH_1x02_P2.50mm_Horizontal" H 10250 5200 50  0001 C CNN
 F 3 "~" H 10250 5200 50  0001 C CNN
 	1    10250 5200
@@
 F 0 "J15" H 9200 7100 50  0000 R CNN
 F 1 "EStop Rly JST2H" H 9550 6900 50  0000 R CNN
-F 2 "Connector_JST:JST_EH_S2B-EH_1x02_P2.50mm_Horizontal" H 9250 7100 50  0001 C CNN
+F 2 "0MiscParts:JST_EH_S2B-EH_1x02_P2.50mm_Horizontal" H 9250 7100 50  0001 C CNN
 F 3 "~" H 9250 7100 50  0001 C CNN
 	1    9250 7100
@@
 F 0 "J16" H 9250 8000 50  0000 R CNN
 F 1 "Sp Rly 1 JST2H" H 9600 7800 50  0000 R CNN
-F 2 "Connector_JST:JST_EH_S2B-EH_1x02_P2.50mm_Horizontal" H 9300 8000 50  0001 C CNN
+F 2 "0MiscParts:JST_EH_S2B-EH_1x02_P2.50mm_Horizontal" H 9300 8000 50  0001 C CNN
 F 3 "~" H 9300 8000 50  0001 C CNN
 	1    9300 8000
@@
 F 0 "J17" H 9250 8850 50  0000 R CNN
 F 1 "Sp Rly 2 JST2H" H 9600 8650 50  0000 R CNN
-F 2 "Connector_JST:JST_EH_S2B-EH_1x02_P2.50mm_Horizontal" H 9300 8850 50  0001 C CNN
+F 2 "0MiscParts:JST_EH_S2B-EH_1x02_P2.50mm_Horizontal" H 9300 8850 50  0001 C CNN
 F 3 "~" H 9300 8850 50  0001 C CNN
 	1    9300 8850
@@
 F 0 "J11" H 6000 10250 50  0000 R CNN
 F 1 "EStop Sig1 JST2H" H 6700 10250 50  0000 R CNN
-F 2 "Connector_JST:JST_EH_S2B-EH_1x02_P2.50mm_Horizontal" H 6150 10100 50  0001 C CNN
+F 2 "0MiscParts:JST_EH_S2B-EH_1x02_P2.50mm_Horizontal" H 6150 10100 50  0001 C CNN
 F 3 "~" H 6150 10100 50  0001 C CNN
 	1    6150 10100
@@
 F 0 "J18" H 9850 10050 50  0000 R CNN
 F 1 "Step Disable JST2H" H 10400 10200 50  0000 R CNN
-F 2 "Connector_JST:JST_EH_S2B-EH_1x02_P2.50mm_Horizontal" H 9900 10050 50  0001 C CNN
+F 2 "0MiscParts:JST_EH_S2B-EH_1x02_P2.50mm_Horizontal" H 9900 10050 50  0001 C CNN
 F 3 "~" H 9900 10050 50  0001 C CNN
 	1    9900 10050
@@
 L Device:R R20
 U 1 1 608C976B
-P 9200 9500
-F 0 "R20" V 9100 9450 50  0000 C CNN
-F 1 "R" V 9100 9550 50  0000 C CNN
-F 2 "Resistor_SMD:R_0805_2012Metric_Pad1.15x1.40mm_HandSolder" V 9130 9500 50  0001 C CNN
-F 3 "~" H 9200 9500 50  0001 C CNN
-	1    9200 9500
+P 9650 9500
+F 0 "R20" V 9550 9450 50  0000 C CNN
+F 1 "R" V 9550 9550 50  0000 C CNN
+F 2 "Resistor_SMD:R_0805_2012Metric_Pad1.15x1.40mm_HandSolder" V 9580 9500 50  0001 C CNN
+F 3 "~" H 9650 9500 50  0001 C CNN
+	1    9650 9500
 	0    1    1    0
 $EndComp
@@
 L Device:LED D17
 U 1 1 608C9771
-P 9650 9500
-F 0 "D17" H 9500 9600 50  0000 C CNN
-F 1 "LED" H 9650 9600 50  0000 C CNN
-F 2 "LED_SMD:LED_0805_2012Metric_Pad1.15x1.40mm_HandSolder" H 9650 9500 50  0001 C CNN
-F 3 "~" H 9650 9500 50  0001 C CNN
-	1    9650 9500
+P 9200 9500
+F 0 "D17" H 9050 9600 50  0000 C CNN
+F 1 "LED" H 9200 9600 50  0000 C CNN
+F 2 "LED_SMD:LED_0805_2012Metric_Pad1.15x1.40mm_HandSolder" H 9200 9500 50  0001 C CNN
+F 3 "~" H 9200 9500 50  0001 C CNN
+	1    9200 9500
 	1    0    0    -1
 $EndComp
@@
 L Device:C C7
 U 1 1 60B24430
-P 6250 5350
-F 0 "C7" H 6365 5396 50  0000 L CNN
-F 1 ".1uf" H 6365 5305 50  0000 L CNN
-F 2 "Capacitor_SMD:C_0805_2012Metric_Pad1.15x1.40mm_HandSolder" H 6288 5200 50  0001 C CNN
-F 3 "~" H 6250 5350 50  0001 C CNN
-	1    6250 5350
+P 10450 9850
+F 0 "C7" H 10565 9896 50  0000 L CNN
+F 1 ".1uf" H 10565 9805 50  0000 L CNN
+F 2 "Capacitor_SMD:C_0805_2012Metric_Pad1.15x1.40mm_HandSolder" H 10488 9700 50  0001 C CNN
+F 3 "~" H 10450 9850 50  0001 C CNN
+	1    10450 9850
 	1    0    0    -1
 $EndComp
@@
 L power:GND #PWR044
 U 1 1 60B24436
-P 6250 5500
-F 0 "#PWR044" H 6250 5250 50  0001 C CNN
-F 1 "GND" H 6255 5327 50  0000 C CNN
-F 2 "" H 6250 5500 50  0001 C CNN
-F 3 "" H 6250 5500 50  0001 C CNN
-	1    6250 5500
+P 10450 10000
+F 0 "#PWR044" H 10450 9750 50  0001 C CNN
+F 1 "GND" H 10455 9827 50  0000 C CNN
+F 2 "" H 10450 10000 50  0001 C CNN
+F 3 "" H 10450 10000 50  0001 C CNN
+	1    10450 10000
 	1    0    0    -1
 $EndComp
@@
 L power:+5V #PWR043
 U 1 1 60B2443C
-P 6250 5200
-F 0 "#PWR043" H 6250 5050 50  0001 C CNN
-F 1 "+5V" H 6265 5373 50  0000 C CNN
-F 2 "" H 6250 5200 50  0001 C CNN
-F 3 "" H 6250 5200 50  0001 C CNN
-	1    6250 5200
-	1    0    0    -1
-$EndComp
-$Comp
-L Device:C C8
-U 1 1 60B3AADD
-P 6700 5350
-F 0 "C8" H 6815 5396 50  0000 L CNN
-F 1 ".1uf" H 6815 5305 50  0000 L CNN
-F 2 "Capacitor_SMD:C_0805_2012Metric_Pad1.15x1.40mm_HandSolder" H 6738 5200 50  0001 C CNN
-F 3 "~" H 6700 5350 50  0001 C CNN
-	1    6700 5350
-	1    0    0    -1
-$EndComp
-$Comp
-L power:GND #PWR047
-U 1 1 60B3AAE3
-P 6700 5500
-F 0 "#PWR047" H 6700 5250 50  0001 C CNN
-F 1 "GND" H 6705 5327 50  0000 C CNN
-F 2 "" H 6700 5500 50  0001 C CNN
-F 3 "" H 6700 5500 50  0001 C CNN
-	1    6700 5500
-	1    0    0    -1
-$EndComp
-$Comp
-L power:+5V #PWR046
-U 1 1 60B3AAE9
-P 6700 5200
-F 0 "#PWR046" H 6700 5050 50  0001 C CNN
-F 1 "+5V" H 6715 5373 50  0000 C CNN
-F 2 "" H 6700 5200 50  0001 C CNN
-F 3 "" H 6700 5200 50  0001 C CNN
-	1    6700 5200
+P 10450 9700
+F 0 "#PWR043" H 10450 9550 50  0001 C CNN
+F 1 "+5V" H 10465 9873 50  0000 C CNN
+F 2 "" H 10450 9700 50  0001 C CNN
+F 3 "" H 10450 9700 50  0001 C CNN
+	1    10450 9700
 	1    0    0    -1
 $EndComp
@@
 F 0 "J26" H 16600 2950 50  0000 R CNN
 F 1 "VFD Dir JST3H" H 16750 3050 50  0000 R CNN
-F 2 "Connector_JST:JST_EH_S3B-EH_1x03_P2.50mm_Horizontal" H 16250 3300 50  0001 C CNN
+F 2 "0MiscParts:JST_EH_S3B-EH_1x03_P2.50mm_Horizontal" H 16250 3300 50  0001 C CNN
 F 3 "~" H 16250 3300 50  0001 C CNN
 	1    16250 3300
@@
 F 0 "J27" H 16750 6700 50  0000 R CNN
 F 1 "VFD Ctl JST3H" H 16900 6600 50  0000 R CNN
-F 2 "Connector_JST:JST_EH_S3B-EH_1x03_P2.50mm_Horizontal" H 16350 6350 50  0001 C CNN
+F 2 "0MiscParts:JST_EH_S3B-EH_1x03_P2.50mm_Horizontal" H 16350 6350 50  0001 C CNN
 F 3 "~" H 16350 6350 50  0001 C CNN
 	1    16350 6350
@@
 F 0 "J23" H 14800 8850 50  0000 R CNN
 F 1 "Sw 12v 1 JST2H" H 15200 8650 50  0000 R CNN
-F 2 "Connector_JST:JST_EH_S2B-EH_1x02_P2.50mm_Horizontal" H 14900 8850 50  0001 C CNN
+F 2 "0MiscParts:JST_EH_S2B-EH_1x02_P2.50mm_Horizontal" H 14900 8850 50  0001 C CNN
 F 3 "~" H 14900 8850 50  0001 C CNN
 	1    14900 8850
@@
 F 0 "J24" H 14800 9700 50  0000 R CNN
 F 1 "Sw 12v 2 JST2H" H 15200 9500 50  0000 R CNN
-F 2 "Connector_JST:JST_EH_S2B-EH_1x02_P2.50mm_Horizontal" H 14900 9700 50  0001 C CNN
+F 2 "0MiscParts:JST_EH_S2B-EH_1x02_P2.50mm_Horizontal" H 14900 9700 50  0001 C CNN
 F 3 "~" H 14900 9700 50  0001 C CNN
 	1    14900 9700
@@
 F 0 "J25" H 16300 1000 50  0000 R CNN
 F 1 "Pilot JST2H" H 16650 700 50  0000 R CNN
-F 2 "Connector_JST:JST_EH_S2B-EH_1x02_P2.50mm_Horizontal" H 16250 900 50  0001 C CNN
+F 2 "0MiscParts:JST_EH_S2B-EH_1x02_P2.50mm_Horizontal" H 16250 900 50  0001 C CNN
 F 3 "~" H 16250 900 50  0001 C CNN
 	1    16250 900
@@
 EStopRlyOut
 Text Label 8350 7200 0    50   ~ 0
-EStopRlyDrv
+EStopRlyExt
 Text Label 7150 9650 0    50   ~ 0
 StepDisOut
@@
 Sp1R
 Text Label 8700 6900 0    50   ~ 0
-ESR
+ESRR
 Text Label 8700 6400 0    50   ~ 0
-EGR
+ESSR
 $Comp
 L Device:R R10

Commit message: Add labels to silk screen.
Parts:
- renumbered C11 to C10, C12 to C11, C13 to C12, C14 to C13, C15 to C14, C9 to C8, C10 to C9
Other:
- moved on the sheet: C7

Commit message: Designed front panel.  More updates to output.
Parts:
- removed K1, K2, K3: G6S-2, Relay_THT:Relay_DPDT_Omron_G6S-2, symbol Relay:G6S-2
- removed U4: 74LVC2G00, Package_SO:TSSOP-8_3x3mm_P0.65mm, symbol 74xGxx:74LVC2G00
- added D9: D_Zener_x2_ACom_KKA, 0MiscParts:SOT-23-Handsoldering, symbol Device:D_Zener_x2_ACom_KKA
- added K1, K2, K3: G6S-2, 0MiscParts:Relay_DPDT_Omron_G6S-2, symbol 00User:G6S-2
- added R13, R14, R25: 10k, Resistor_SMD:R_0805_2012Metric_Pad1.15x1.40mm_HandSolder, symbol Device:R
- added R17: 200, Resistor_SMD:R_0805_2012Metric_Pad1.15x1.40mm_HandSolder, symbol Device:R
- added U4: 74LVC1G08, Package_TO_SOT_SMD:SOT-23-5, symbol 74xGxx:74LVC1G08
- J1: value Control -> Control JST5H
- J11: value EStop Sig1 JST2H -> Ext Step Disable JST2H
- J13: value JTAG -> JTAG 2x05
- J14: value Dbg -> Dbg 2x03
- J4: value TmrTest -> TmrTest 1x03
- J5: value DbgPort -> DbgPort JST4H
- J6: value RemPort -> RemPort JST3H
- J7: value 12VIn -> 12VIn JST2H
- J8: value PwrIn -> PwrIn JST2H
- R24: renamed from R15; value R -> 10k
- renumbered D9 to D10, D10 to D11, D11 to D12, D12 to D13, D17 to D14, D13 to D15, D14 to D16, D15 to D17, D16 to D18, D18 to D19, D19 to D20, D20 to D21, D21 to D22, D22 to D23, D23 to D24, D24 to D25, D25 to D26, J25 to J23, J23 to J24, J24 to J25, R13 to R15, R14 to R16, R16 to R18, R17 to R19, R18 to R20, R19 to R21, R20 to R22, R21 to R23, R22 to R26, R23 to R27, R24 to R28, R25 to R29, R26 to R30, R27 to R31, R33 to R32, R28 to R33, R29 to R34, R30 to R35, R31 to R36, R32 to R37
Connections:
- net labels added: ProcSpdlRly1, ProcSpdlRly2, StepDisIn
- net labels removed: ProcSpindleRly, StepDisOut
- wire segments 408 -> 421
Other:
- moved on the sheet: C7, D10, D11, D12, D13, D14, D15, D16, D17, D18, D5, J10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

Commit message: Add ferrite and capacitor to filter VFD control voltage.
Parts:
- added C15: .1uf, Capacitor_SMD:C_0805_2012Metric_Pad1.15x1.40mm_HandSolder, symbol Device:C
- added FB1: Ferrite_Bead, Inductor_SMD:L_0805_2012Metric_Pad1.15x1.40mm_HandSolder, symbol Device:Ferrite_Bead
- renumbered C14 to C12, C12 to C13, C13 to C14
Connections:
- net labels added: MaxV, MaxVFilt
- net labels removed: RefIn
- wire segments 421 -> 423
Other:
- moved on the sheet: C12, U10C

Commit message: Boards sent to be built.
Parts:
- removed U4: 74LVC1G08, Package_TO_SOT_SMD:SOT-23-5, symbol 74xGxx:74LVC1G08
- added JP5: SolderJumper_3_Open, 0MiscParts:Jumper_0603_3, symbol Jumper:SolderJumper_3_Open
- added R38: R, Resistor_SMD:R_0805_2012Metric_Pad1.15x1.40mm_HandSolder, symbol Device:R
- added U11: LM4040DBZ-10, 0MiscParts:SOT-23-Handsoldering, symbol Reference_Voltage:LM4040DBZ-10
- added U4: 74LVC1G00, Package_TO_SOT_SMD:SOT-23-5, symbol 74xGxx:74LVC1G00
Connections:
- net labels added: IntRef
- wire segments 423 -> 429
Other:
- note added: "StepDis=1 when WDOut=0\nor ProcStepDis=0"
Changed lines of the file:
@@
 P 7300 9000
 F 0 "#PWR048" H 7300 8850 50  0001 C CNN
-F 1 "+5V" H 7300 9200 50  0000 C CNN
+F 1 "+5V" H 7450 9100 50  0000 C CNN
 F 2 "" H 7300 9000 50  0001 C CNN
 F 3 "" H 7300 9000 50  0001 C CNN
@@
 $EndComp
 $Comp
-L power:GND #PWR0114
+L power:GND #PWR0115
 U 1 1 60CD8BBF
 P 13800 3000
-F 0 "#PWR0114" H 13800 2750 50  0001 C CNN
+F 0 "#PWR0115" H 13800 2750 50  0001 C CNN
 F 1 "GND" H 13805 2827 50  0000 C CNN
 F 2 "" H 13800 3000 50  0001 C CNN
@@
 $EndComp
 $Comp
-L power:GND #PWR0134
+L power:GND #PWR0136
 U 1 1 60E8C10C
 P 16100 6500
-F 0 "#PWR0134" H 16100 6250 50  0001 C CNN
+F 0 "#PWR0136" H 16100 6250 50  0001 C CNN
 F 1 "GND" H 16105 6327 50  0000 C CNN
 F 2 "" H 16100 6500 50  0001 C CNN
@@
 	14050 6000 14050 5900
 $Comp
-L power:GND #PWR0116
+L power:GND #PWR0117
 U 1 1 61056637
 P 14050 6300
-F 0 "#PWR0116" H 14050 6050 50  0001 C CNN
+F 0 "#PWR0117" H 14050 6050 50  0001 C CNN
 F 1 "GND" H 14055 6127 50  0000 C CNN
 F 2 "" H 14050 6300 50  0001 C CNN
@@
 	1    0    0    -1
 $EndComp
-Text Label 15300 6000 0    50   ~ 0
-MaxVFilt
 Text Label 15350 6750 0    50   ~ 0
 CtlV
@@
 MaxV
 $Comp
-L power:GND #PWR0113
+L power:GND #PWR0114
 U 1 1 6110B294
 P 13750 7850
-F 0 "#PWR0113" H 13750 7600 50  0001 C CNN
+F 0 "#PWR0114" H 13750 7600 50  0001 C CNN
 F 1 "GND" H 13755 7677 50  0000 C CNN
 F 2 "" H 13750 7850 50  0001 C CNN
@@
 $EndComp
 $Comp
-L power:+12V #PWR0120
+L power:+12V #PWR0113
 U 1 1 61129A23
 P 13750 7250
-F 0 "#PWR0120" H 13750 7100 50  0001 C CNN
+F 0 "#PWR0113" H 13750 7100 50  0001 C CNN
 F 1 "+12V" H 13765 7423 50  0000 C CNN
 F 2 "" H 13750 7250 50  0001 C CNN
@@
 $EndComp
 $Comp
-L power:GND #PWR0117
+L power:GND #PWR0118
 U 1 1 6112A61D
 P 14150 7250
-F 0 "#PWR0117" H 14150 7000 50  0001 C CNN
+F 0 "#PWR0118" H 14150 7000 50  0001 C CNN
 F 1 "GND" H 14155 7077 50  0000 C CNN
 F 2 "" H 14150 7250 50  0001 C CNN
@@
 $EndComp
 $Comp
-L power:GND #PWR0115
+L power:GND #PWR0116
 U 1 1 61251EE9
 P 13800 5000
-F 0 "#PWR0115" H 13800 4750 50  0001 C CNN
+F 0 "#PWR0116" H 13800 4750 50  0001 C CNN
 F 1 "GND" H 13805 4827 50  0000 C CNN
 F 2 "" H 13800 5000 50  0001 C CNN
@@
 	13900 8950 13900 8650
 $Comp
-L power:+12V #PWR0118
+L power:+12V #PWR0119
 U 1 1 6179EE05
 P 14700 8850
-F 0 "#PWR0118" H 14700 8700 50  0001 C CNN
+F 0 "#PWR0119" H 14700 8700 50  0001 C CNN
 F 1 "+12V" V 14715 8978 50  0000 L CNN
 F 2 "" H 14700 8850 50  0001 C CNN
@@
 	13900 9800 13900 9500
 $Comp
-L power:+12V #PWR0119
+L power:+12V #PWR0120
 U 1 1 6181213A
 P 14700 9700
-F 0 "#PWR0119" H 14700 9550 50  0001 C CNN
+F 0 "#PWR0120" H 14700 9550 50  0001 C CNN
 F 1 "+12V" V 14715 9828 50  0000 L CNN
 F 2 "" H 14700 9700 50  0001 C CNN
@@
 Wire Wire Line
 	6100 3800 5600 3800
-$Comp
-L 74xGxx:74LVC1G08 U4
-U 1 1 6536F774
-P 7300 9100
-F 0 "U4" H 7450 9300 50  0000 C CNN
-F 1 "74LVC1G08" H 7000 9300 50  0000 C CNN
-F 2 "Package_TO_SOT_SMD:SOT-23-5" H 7300 9100 50  0001 C CNN
-F 3 "http://www.ti.com/lit/sg/scyt129e/scyt129e.pdf" H 7300 9100 50  0001 C CNN
-	1    7300 9100
-	1    0    0    -1
-$EndComp
 Wire Wire Line
 	8750 10000 9300 10000
@@
 $EndComp
 Wire Wire Line
-	15900 7200 16350 7200
+	15900 7200 16250 7200
 Text Label 16000 7200 0    50   ~ 0
 MaxV
@@
 	0    1    1    0
 $EndComp
-Wire Wire Line
-	15150 7200 15600 7200
 Text Label 15200 7200 0    50   ~ 0
 MaxVFilt
 Connection ~ 15600 7200
+Text Notes 10150 9000 0    50   ~ 0
+StepDis=1 when WDOut=0\nor ProcStepDis=0
+$Comp
+L 74xGxx:74LVC1G00 U4
+U 1 1 65D9995D
+P 7300 9100
+F 0 "U4" H 7275 9367 50  0000 C CNN
+F 1 "74LVC1G00" H 7000 9300 50  0000 C CNN
+F 2 "Package_TO_SOT_SMD:SOT-23-5" H 7300 9100 50  0001 C CNN
+F 3 "http://www.ti.com/lit/sg/scyt129e/scyt129e.pdf" H 7300 9100 50  0001 C CNN
+	1    7300 9100
+	1    0    0    -1
+$EndComp
+$Comp
+L Reference_Voltage:LM4040DBZ-10 U11
+U 1 1 6000DA5A
+P 15950 8050
+F 0 "U11" V 15996 7962 50  0000 R CNN
+F 1 "LM4040DBZ-10" V 15900 8750 50  0000 R CNN
+F 2 "0MiscParts:SOT-23-Handsoldering" H 15950 7850 50  0001 C CIN
+F 3 "http://www.ti.com/lit/ds/symlink/lm4040-n.pdf" H 15950 8050 50  0001 C CIN
+	1    15950 8050
+	0    -1   -1   0
+$EndComp
+$Comp
+L power:GND #PWR0135
+U 1 1 6001016A
+P 15950 8200
+F 0 "#PWR0135" H 15950 7950 50  0001 C CNN
+F 1 "GND" H 15955 8027 50  0000 C CNN
+F 2 "" H 15950 8200 50  0001 C CNN
+F 3 "" H 15950 8200 50  0001 C CNN
+	1    15950 8200
+	1    0    0    -1
+$EndComp
+$Comp
+L Device:R R38
+U 1 1 600104DE
+P 15950 7650
+F 0 "R38" V 15850 7600 50  0000 C CNN
+F 1 "R" V 15850 7700 50  0000 C CNN
+F 2 "Resistor_SMD:R_0805_2012Metric_Pad1.15x1.40mm_HandSolder" V 15880 7650 50  0001 C CNN
+F 3 "~" H 15950 7650 50  0001 C CNN
+	1    15950 7650
+	-1   0    0    1
+$EndComp
+$Comp
+L power:+12V #PWR0134
+U 1 1 60049A67
+P 15950 7500
+F 0 "#PWR0134" H 15950 7350 50  0001 C CNN
+F 1 "+12V" H 15965 7673 50  0000 C CNN
+F 2 "" H 15950 7500 50  0001 C CNN
+F 3 "" H 15950 7500 50  0001 C CNN
+	1    15950 7500
+	1    0    0    -1
+$EndComp
+Wire Wire Line
+	15950 7900 15950 7850
+$Comp
+L Jumper:SolderJumper_3_Open JP5
+U 1 1 60083FA7
+P 14950 7550
+F 0 "JP5" V 14996 7618 50  0000 L CNN
+F 1 "SolderJumper_3_Open" V 14550 7150 50  0000 L CNN
+F 2 "0MiscParts:Jumper_0603_3" H 14950 7550 50  0001 C CNN
+F 3 "~" H 14950 7550 50  0001 C CNN
+	1    14950 7550
+	0    1    -1   0
+$EndComp
+Wire Wire Line
+	15950 7850 14950 7850
+Connection ~ 15950 7850
+Wire Wire Line
+	15950 7850 15950 7800
+Wire Wire Line
+	14950 7350 14950 7200
+Wire Wire Line
+	14950 7200 15600 7200
+Wire Wire Line
+	14500 7550 14800 7550
+Text Label 15200 7850 0    50   ~ 0
+IntRef
+Text Label 14550 7550 0    50   ~ 0
+PWMRef
+Text Label 15200 6000 0    50   ~ 0
+PWMRef
+Wire Wire Line
+	14950 7850 14950 7750
 $EndSCHEMATC
