File: OutputMega/OutputMega.sch (KiCad schematic (older format))
At the start: 143 parts, among them J1 Control JST5H, J10 Conn_02x13_Top_Bottom, J11 Ext Step Disable JST2H, J12 MegaProMiniR, J13 JTAG 2x05, J14 Dbg 2x03, J15 EStop Rly JST2H, J16 Sp Rly 1 JST2H, J17 Sp Rly 2 JST2H, J18 Step Disable JST2H, J19 EStop Sig0 JST2H, J2 EStop JST3H, J20 EStop Sig1 JST2H, J21 Conn_01x06_Male, J22 Conn_02x05_Odd_Even, J23 Pilot JST2H, J24 Sw 12v 1 JST2H, J25 Sw 12v 2 JST2H, J26 VFD Dir JST3H, J27 VFD Ctl JST3H, J3 EStop Rst JST2H, J4 TmrTest 1x03, J5 DbgPort JST4H, J6 RemPort JST3H, J7 12VIn JST2H, J8 PwrIn JST2H, J9 MegaProMiniL, K1 G6S-2, K2 G6S-2, K3 G6S-2, Q1 2N7002, Q10 2N7002, Q11 2N7002, Q12 2N7002, Q13 2N7002, Q2 2N7002, Q3 2N7002, Q4 2N7002, Q5 2N7002, Q6 2N7002, Q7 2N7002, Q8 2N7002, Q9 2N7002, U1 74HCT123, U10 MC34072AP, U11 LM4040DBZ-10, U2 74LS08, U3 LD1117S50TR_SOT223, U4 74LVC1G00, U5 74AUC2G34, U6 74AUC2G34, U7 74LVC2G157, U8 74LS08, U9 TLV9351

Commit message: Updates for new boards.
Parts:
- C6: value C -> 10uf
- R16, R22: value R -> 7.5k
- R18, R19, R20, R21, R34, R35, R36, R37, R8: value R -> 24k
- R23: value R -> 2.4k
- R26, R27, R28, R29: value R -> 10k
- R32: value R -> 750
- R38: value R -> 1k
Changed lines of the file:
@@
 P 3150 900
 F 0 "R8" H 3220 946 50  0000 L CNN
-F 1 "R" H 3220 855 50  0000 L CNN
+F 1 "24k" H 3220 855 50  0000 L CNN
 F 2 "Resistor_SMD:R_0805_2012Metric_Pad1.15x1.40mm_HandSolder" V 3080 900 50  0001 C CNN
 F 3 "~" H 3150 900 50  0001 C CNN
@@
 P 6050 950
 F 0 "R16" H 6120 996 50  0000 L CNN
-F 1 "R" H 6120 905 50  0000 L CNN
+F 1 "7.5k" H 6120 905 50  0000 L CNN
 F 2 "Resistor_SMD:R_0805_2012Metric_Pad1.15x1.40mm_HandSolder" V 5980 950 50  0001 C CNN
 F 3 "~" H 6050 950 50  0001 C CNN
@@
 P 5550 1150
 F 0 "C6" H 5665 1196 50  0000 L CNN
-F 1 "C" H 5665 1105 50  0000 L CNN
+F 1 "10uf" H 5665 1105 50  0000 L CNN
 F 2 "Capacitor_SMD:C_0805_2012Metric_Pad1.15x1.40mm_HandSolder" H 5588 1000 50  0001 C CNN
 F 3 "~" H 5550 1150 50  0001 C CNN
@@
 U 1 1 603F0247
 P 9350 6000
-F 0 "R18" V 9250 5950 50  0000 C CNN
-F 1 "R" V 9250 6050 50  0000 C CNN
+F 0 "R18" V 9250 6000 50  0000 C CNN
+F 1 "24k" V 9350 6000 50  0000 C CNN
 F 2 "Resistor_SMD:R_0805_2012Metric_Pad1.15x1.40mm_HandSolder" V 9280 6000 50  0001 C CNN
 F 3 "~" H 9350 6000 50  0001 C CNN
@@
 U 1 1 6062B080
 P 9350 6500
-F 0 "R19" V 9250 6450 50  0000 C CNN
-F 1 "R" V 9250 6550 50  0000 C CNN
+F 0 "R19" V 9250 6500 50  0000 C CNN
+F 1 "24k" V 9350 6500 50  0000 C CNN
 F 2 "Resistor_SMD:R_0805_2012Metric_Pad1.15x1.40mm_HandSolder" V 9280 6500 50  0001 C CNN
 F 3 "~" H 9350 6500 50  0001 C CNN
@@
 U 1 1 6073FC7E
 P 9400 7400
-F 0 "R20" V 9300 7350 50  0000 C CNN
-F 1 "R" V 9300 7450 50  0000 C CNN
+F 0 "R20" V 9300 7400 50  0000 C CNN
+F 1 "24k" V 9400 7400 50  0000 C CNN
 F 2 "Resistor_SMD:R_0805_2012Metric_Pad1.15x1.40mm_HandSolder" V 9330 7400 50  0001 C CNN
 F 3 "~" H 9400 7400 50  0001 C CNN
@@
 U 1 1 607556BB
 P 9400 8250
-F 0 "R21" V 9300 8200 50  0000 C CNN
-F 1 "R" V 9300 8300 50  0000 C CNN
+F 0 "R21" V 9300 8250 50  0000 C CNN
+F 1 "24k" V 9400 8250 50  0000 C CNN
 F 2 "Resistor_SMD:R_0805_2012Metric_Pad1.15x1.40mm_HandSolder" V 9330 8250 50  0001 C CNN
 F 3 "~" H 9400 8250 50  0001 C CNN
@@
 U 1 1 608C976B
 P 9450 8900
-F 0 "R22" V 9350 8850 50  0000 C CNN
-F 1 "R" V 9350 8950 50  0000 C CNN
+F 0 "R22" V 9350 8900 50  0000 C CNN
+F 1 "7.5k" V 9450 8900 50  0000 C CNN
 F 2 "Resistor_SMD:R_0805_2012Metric_Pad1.15x1.40mm_HandSolder" V 9380 8900 50  0001 C CNN
 F 3 "~" H 9450 8900 50  0001 C CNN
@@
 U 1 1 60936ACD
 P 9450 9150
-F 0 "R23" V 9350 9100 50  0000 C CNN
-F 1 "R" V 9350 9200 50  0000 C CNN
+F 0 "R23" V 9350 9150 50  0000 C CNN
+F 1 "2.4k" V 9450 9150 50  0000 C CNN
 F 2 "Resistor_SMD:R_0805_2012Metric_Pad1.15x1.40mm_HandSolder" V 9380 9150 50  0001 C CNN
 F 3 "~" H 9450 9150 50  0001 C CNN
@@
 U 1 1 60CD8BD3
 P 14850 3000
-F 0 "R36" V 14750 2950 50  0000 C CNN
-F 1 "R" V 14750 3050 50  0000 C CNN
+F 0 "R36" V 14750 3000 50  0000 C CNN
+F 1 "24k" V 14850 3000 50  0000 C CNN
 F 2 "Resistor_SMD:R_0805_2012Metric_Pad1.15x1.40mm_HandSolder" V 14780 3000 50  0001 C CNN
 F 3 "~" H 14850 3000 50  0001 C CNN
@@
 U 1 1 61251EFD
 P 14850 5000
-F 0 "R37" V 14750 4950 50  0000 C CNN
-F 1 "R" V 14750 5050 50  0000 C CNN
+F 0 "R37" V 14750 5000 50  0000 C CNN
+F 1 "24k" V 14850 5000 50  0000 C CNN
 F 2 "Resistor_SMD:R_0805_2012Metric_Pad1.15x1.40mm_HandSolder" V 14780 5000 50  0001 C CNN
 F 3 "~" H 14850 5000 50  0001 C CNN
@@
 U 1 1 615A767A
 P 12600 5250
-F 0 "R28" V 12500 5200 50  0000 C CNN
-F 1 "R" V 12500 5300 50  0000 C CNN
+F 0 "R28" V 12500 5250 50  0000 C CNN
+F 1 "10k" V 12600 5250 50  0000 C CNN
 F 2 "Resistor_SMD:R_0805_2012Metric_Pad1.15x1.40mm_HandSolder" V 12530 5250 50  0001 C CNN
 F 3 "~" H 12600 5250 50  0001 C CNN
@@
 U 1 1 615C7851
 P 12600 5450
-F 0 "R29" V 12500 5400 50  0000 C CNN
-F 1 "R" V 12500 5500 50  0000 C CNN
+F 0 "R29" V 12500 5450 50  0000 C CNN
+F 1 "10k" V 12600 5450 50  0000 C CNN
 F 2 "Resistor_SMD:R_0805_2012Metric_Pad1.15x1.40mm_HandSolder" V 12530 5450 50  0001 C CNN
 F 3 "~" H 12600 5450 50  0001 C CNN
@@
 U 1 1 616CC3D1
 P 12400 9900
-F 0 "R26" V 12300 9850 50  0000 C CNN
-F 1 "R" V 12300 9950 50  0000 C CNN
+F 0 "R26" V 12300 9900 50  0000 C CNN
+F 1 "10k" V 12400 9900 50  0000 C CNN
 F 2 "Resistor_SMD:R_0805_2012Metric_Pad1.15x1.40mm_HandSolder" V 12330 9900 50  0001 C CNN
 F 3 "~" H 12400 9900 50  0001 C CNN
@@
 U 1 1 616CC3D8
 P 12400 10100
-F 0 "R27" V 12300 10050 50  0000 C CNN
-F 1 "R" V 12300 10150 50  0000 C CNN
+F 0 "R27" V 12300 10100 50  0000 C CNN
+F 1 "10k" V 12400 10100 50  0000 C CNN
 F 2 "Resistor_SMD:R_0805_2012Metric_Pad1.15x1.40mm_HandSolder" V 12330 10100 50  0001 C CNN
 F 3 "~" H 12400 10100 50  0001 C CNN
@@
 U 1 1 61778FEF
 P 14650 8650
-F 0 "R34" V 14550 8600 50  0000 C CNN
-F 1 "R" V 14550 8700 50  0000 C CNN
+F 0 "R34" V 14550 8650 50  0000 C CNN
+F 1 "24k" V 14650 8650 50  0000 C CNN
 F 2 "Resistor_SMD:R_0805_2012Metric_Pad1.15x1.40mm_HandSolder" V 14580 8650 50  0001 C CNN
 F 3 "~" H 14650 8650 50  0001 C CNN
@@
 U 1 1 61812122
 P 14650 9500
-F 0 "R35" V 14550 9450 50  0000 C CNN
-F 1 "R" V 14550 9550 50  0000 C CNN
+F 0 "R35" V 14550 9500 50  0000 C CNN
+F 1 "24k" V 14650 9500 50  0000 C CNN
 F 2 "Resistor_SMD:R_0805_2012Metric_Pad1.15x1.40mm_HandSolder" V 14580 9500 50  0001 C CNN
 F 3 "~" H 14650 9500 50  0001 C CNN
@@
 U 1 1 62898919
 P 13600 850
-F 0 "R32" V 13500 800 50  0000 C CNN
-F 1 "R" V 13500 900 50  0000 C CNN
+F 0 "R32" V 13500 850 50  0000 C CNN
+F 1 "750" V 13600 850 50  0000 C CNN
 F 2 "Resistor_SMD:R_0805_2012Metric_Pad1.15x1.40mm_HandSolder" V 13530 850 50  0001 C CNN
 F 3 "~" H 13600 850 50  0001 C CNN
@@
 U 1 1 600104DE
 P 15950 7650
-F 0 "R38" V 15850 7600 50  0000 C CNN
-F 1 "R" V 15850 7700 50  0000 C CNN
+F 0 "R38" H 15800 7600 50  0000 C CNN
+F 1 "1k" H 15800 7700 50  0000 C CNN
 F 2 "Resistor_SMD:R_0805_2012Metric_Pad1.15x1.40mm_HandSolder" V 15880 7650 50  0001 C CNN
 F 3 "~" H 15950 7650 50  0001 C CNN
