File: Sensor/RTDMount/RTDMount.kicad_pcb (KiCad board)
At the start: 2 copper layers, 15.9 x 11.4 mm, 6 parts, among them J1 Conn_01x03_Male, J2 Conn_01x01_Male, J3 Conn_01x01_Male, J4 Conn_01x01_Male

Commit message: FT4232 Board and some fixes/
Routing:
- added copper zone on B.Cu, net (none)
Changed lines of the file:
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@@
     (last_trace_width 0.254)
     (trace_clearance 0.2032)
-    (zone_clearance 0.508)
+    (zone_clearance 0.254)
     (zone_45_only no)
     (trace_min 0.2)
@@
   (via (at 145.7325 86.6775) (size 0.762) (drill 0.381) (layers F.Cu B.Cu) (net 2))
   (segment (start 145.7325 86.6775) (end 144.9425 87.4675) (width 0.254) (layer F.Cu) (net 2))
+  (zone (net 0) (net_name "") (layer B.Cu) (hatch edge 0.508)
+    (connect_pads (clearance 0.254))
+    (min_thickness 0.254)
+    (fill yes (arc_segments 32) (thermal_gap 0.508) (thermal_bridge_width 0.508))
+    (polygon
+      (pts
+        (xy 154.94 92.71) (xy 137.795 92.71) (xy 137.795 80.01) (xy 154.94 80.01)
+      )
+    )
+  )
 )

Commit message: Updates for new boards.
Parts:
- added J5: Pad, 0MiscParts:SurfaceMountPad, B.Cu at (140.0, 84.8)
- added J6: Pad, 0MiscParts:SurfaceMountPad, F.Cu at (140.0, 84.8)
Routing:
- net /Pad: vias 0 -> 5
- added copper zone on B.Cu, net /Pad
- added copper zone on F.Cu, net /Pad
- removed copper zone on B.Cu, net (none)
Changed lines of the file:
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@@
     (thickness 1.6)
     (drawings 6)
-    (tracks 15)
+    (tracks 20)
     (zones 0)
-    (modules 6)
-    (nets 3)
+    (modules 8)
+    (nets 4)
   )
   (page A4)
@@
     (39 F.Mask user)
     (40 Dwgs.User user)
-    (41 Cmts.User user)
+    (41 Cmts.User user hide)
     (42 Eco1.User user)
     (43 Eco2.User user)
@@
   (net 1 /B)
   (net 2 /A)
+  (net 3 /Pad)
   (net_class Default "This is the default net class."
     (clearance 0.2032)
@@
     (add_net /A)
     (add_net /B)
+    (add_net /Pad)
+  )
+  (module 0MiscParts:SurfaceMountPad (layer F.Cu)
+    (at 139.954 84.7725)
+    (fp_text reference J6 (at 0 -2.5) (layer F.SilkS) hide
+      (effects (font (size 1 1) (thickness 0.15)))
+    )
+    (fp_text value Pad (at 0 -4.2) (layer F.Fab)
+      (effects (font (size 1 1) (thickness 0.15)))
+    )
+    (pad 1 smd rect (at 0 0) (size 1 1) (layers F.Cu F.Paste F.Mask)
+      (net 3 /Pad))
+  )
+  (module 0MiscParts:SurfaceMountPad (layer B.Cu)
+    (at 139.954 84.7725)
+    (fp_text reference J5 (at 0 2.5) (layer B.SilkS) hide
+      (effects (font (size 1 1) (thickness 0.15)) (justify mirror))
+    )
+    (fp_text value Pad (at 0 4.2) (layer B.Fab)
+      (effects (font (size 1 1) (thickness 0.15)) (justify mirror))
+    )
+    (pad 1 smd rect (at 0 0) (size 1 1) (layers B.Cu B.Paste B.Mask)
+      (net 3 /Pad))
   )
   (module 0MiscParts:RectPad-025x100 (layer F.Cu)
@@
   (gr_line (start 138.43 92.075) (end 138.43 80.645) (layer Edge.Cuts) (width 0.05))
   (gr_line (start 154.305 92.075) (end 138.43 92.075) (layer Edge.Cuts) (width 0.05))
+  (via (at 139.9413 84.7725) (size 0.762) (drill 0.381) (layers F.Cu B.Cu) (net 3))
   (segment (start 150.495 88.82) (end 144.86 88.82) (width 0.254) (layer F.Cu) (net 1))
   (segment (start 144.4625 89.2175) (end 140.0175 89.2175) (width 0.254) (layer F.Cu) (net 1))
@@
   (via (at 145.7325 86.6775) (size 0.762) (drill 0.381) (layers F.Cu B.Cu) (net 2))
   (segment (start 145.7325 86.6775) (end 144.9425 87.4675) (width 0.254) (layer F.Cu) (net 2))
-  (zone (net 0) (net_name "") (layer B.Cu) (hatch edge 0.508)
-    (connect_pads (clearance 0.254))
+  (via (at 141.478 88.3412) (size 0.762) (drill 0.381) (layers F.Cu B.Cu) (net 3))
+  (via (at 142.5956 88.3412) (size 0.762) (drill 0.381) (layers F.Cu B.Cu) (net 3))
+  (via (at 139.954 83.566) (size 0.762) (drill 0.381) (layers F.Cu B.Cu) (net 3))
+  (via (at 139.954 85.979) (size 0.762) (drill 0.381) (layers F.Cu B.Cu) (net 3))
+  (zone (net 3) (net_name /Pad) (layer B.Cu) (hatch edge 0.508)
+    (connect_pads yes (clearance 0.254))
     (min_thickness 0.254)
     (fill yes (arc_segments 32) (thermal_gap 0.508) (thermal_bridge_width 0.508))
@@
       )
     )
+  )
+  (zone (net 3) (net_name /Pad) (layer F.Cu) (hatch edge 0.508)
+    (connect_pads yes (clearance 0.254))
+    (min_thickness 0.254)
+    (fill yes (arc_segments 32) (thermal_gap 0.508) (thermal_bridge_width 0.508))
+    (polygon
+      (pts
+        (xy 143.51 92.71) (xy 137.795 92.71) (xy 137.795 80.01) (xy 143.51 80.01)
+      )
+    )
