File: Sensor/RTD/RTD.sch (KiCad schematic (older format))
At the start: 17 parts, among them J1 Conn_02x04_Odd_Even, J2 Conn_01x04_Female, U1 MIC5225, U2 MAX31865

Commit message: Updating component values.  Updates for new Kicad version.
Parts:
- R1: value R -> 400
Changed lines of the file:
@@
 P 7200 3800
 F 0 "R1" H 7270 3846 50  0000 L CNN
-F 1 "R" H 7270 3755 50  0000 L CNN
+F 1 "400" H 7270 3755 50  0000 L CNN
 F 2 "Resistor_SMD:R_0805_2012Metric_Pad1.15x1.40mm_HandSolder" V 7130 3800 50  0001 C CNN
 F 3 "~" H 7200 3800 50  0001 C CNN
