File: LED1/LED1.kicad_pcb (KiCad board)
At the start: 2 copper layers, 41.3 x 22.9 mm, 13 parts, among them J1 Conn_01x02_Female, U1 AL8805

Commit message: Updating component values.  Updates for new Kicad version.
Parts:
- C1: value C -> 2.2uf 25v
- C2: value C -> 1uf
- D1: value D_Schottky -> DFLS240L-7
- L1: value L -> 33uh
- R1: value R -> .300
