File: FT4232/FT4232.kicad_pcb (KiCad board)
At the start: 2 copper layers, 63.5 x 34.9 mm, 66 parts, among them J1 USB_B_Mini, J2 Conn_02x05_Odd_Even, J3 Conn_02x05_Odd_Even, J4 Conn_02x05_Odd_Even, J5 Conn_02x05_Odd_Even, U1 SP6205, U2 93LCxxB, U3 FT4232H, U4 74HC595, Y1 12MHz

Commit message: Updates for new boards.
Parts:
- added D9: LED, 0MiscParts:LED_0603_1608Metric_Pad1.05x1.35mm_HandSolder, F.Cu at (146.3, 100.3)
- added R16: 5.1k, Resistor_SMD:R_0603_1608Metric_Pad1.05x0.95mm_HandSolder, F.Cu at (144.5, 98.4)
- D1, D2, D3, D4, D5, D6, D7, D8: footprint LED_SMD:LED_0603_1608Metric_Pad1.05x0.95mm_HandSolder -> 0MiscParts:LED_0603_1608Metric_Pad1.05x1.35mm_HandSolder
- R3, R4: value 10 -> 10R
- moved C7 0.71 mm to (100.6, 81.9)
- moved R6 0.71 mm to (107.6, 76.2)
- moved U2 0.71 mm to (106.4, 80.0)
- moved R5 0.71 mm to (103.8, 76.2)
- moved C13 0.64 mm to (115.6, 85.7)
- moved C17 0.64 mm to (110.5, 85.7)
- moved Y1 0.64 mm to (113.0, 85.7)
- moved C24 0.08 mm to (141.5, 96.8)
Routing:
- net GND: track 72.4 -> 76.2 mm, vias 20 -> 21
- net /3.3VR: track 0.00 -> 1.91 mm
- net +3V3: track 113.7 -> 114.6 mm
- net /EEData: track 46.3 -> 45.5 mm
- net /VBus: track 10.2 -> 10.9 mm
Other:
- board text added: "3.3v"

Commit message: Updates to component values.
Parts:
- D1, D3, D5, D7, D9: value LED -> LED Gr
- D2, D4, D6, D8: value LED -> LED Yl
- R10, R12, R14, R16, R8: value 5.1k -> 2.4k
- R11, R13, R15, R9: value 5.1k -> 1k
