File: FT4232/FT4232.sch (KiCad schematic (older format))
At the start: 66 parts, among them J1 USB_B_Mini, J2 Conn_02x05_Odd_Even, J3 Conn_02x05_Odd_Even, J4 Conn_02x05_Odd_Even, J5 Conn_02x05_Odd_Even, U1 SP6205, U2 93LCxxB, U3 FT4232H, U4 74HC595, Y1 12MHz

Commit message: Updates for new boards.
Parts:
- added D9: LED, 0MiscParts:LED_0603_1608Metric_Pad1.05x1.35mm_HandSolder, symbol Device:LED
- added R16: 5.1k, Resistor_SMD:R_0603_1608Metric_Pad1.05x0.95mm_HandSolder, symbol Device:R
- D1, D2, D3, D4, D5, D6, D7, D8: footprint LED_SMD:LED_0603_1608Metric_Pad1.05x0.95mm_HandSolder -> 0MiscParts:LED_0603_1608Metric_Pad1.05x1.35mm_HandSolder
- R3, R4: value 10 -> 10R
Connections:
- net labels added: 3.3VR
- wire segments 226 -> 227
Other:
- moved on the sheet: C12
Changed lines of the file:
@@
 P 6000 4750
 F 0 "R3" V 5900 4750 50  0000 C CNN
-F 1 "10" V 6000 4750 50  0000 C CNN
+F 1 "10R" V 6000 4750 50  0000 C CNN
 F 2 "Resistor_SMD:R_0805_2012Metric_Pad1.15x1.40mm_HandSolder" V 5930 4750 50  0001 C CNN
 F 3 "~" H 6000 4750 50  0001 C CNN
@@
 P 6000 4950
 F 0 "R4" V 5900 4950 50  0000 C CNN
-F 1 "10" V 6000 4950 50  0000 C CNN
+F 1 "10R" V 6000 4950 50  0000 C CNN
 F 2 "Resistor_SMD:R_0805_2012Metric_Pad1.15x1.40mm_HandSolder" V 5930 4950 50  0001 C CNN
 F 3 "~" H 6000 4950 50  0001 C CNN
@@
 Connection ~ 6050 8950
 Wire Wire Line
-	6050 8950 7000 8950
-Wire Wire Line
 	6400 9300 6400 8450
 Connection ~ 6400 8450
@@
 L power:GND #PWR022
 U 1 1 6012287C
-P 7200 4500
-F 0 "#PWR022" H 7200 4250 50  0001 C CNN
-F 1 "GND" H 7205 4327 50  0000 C CNN
-F 2 "" H 7200 4500 50  0001 C CNN
-F 3 "" H 7200 4500 50  0001 C CNN
-	1    7200 4500
+P 7100 4500
+F 0 "#PWR022" H 7100 4250 50  0001 C CNN
+F 1 "GND" H 7105 4327 50  0000 C CNN
+F 2 "" H 7100 4500 50  0001 C CNN
+F 3 "" H 7100 4500 50  0001 C CNN
+	1    7100 4500
 	1    0    0    -1
 $EndComp
@@
 $EndComp
 Wire Wire Line
-	7200 4200 7200 4000
+	7100 4200 7100 4000
 Wire Wire Line
 	7550 4200 7550 4000
@@
 L Device:CP C12
 U 1 1 60122890
-P 7200 4350
-F 0 "C12" H 7318 4396 50  0000 L CNN
-F 1 "4.7uf" H 7318 4305 50  0000 L CNN
-F 2 "Capacitor_Tantalum_SMD:CP_EIA-3216-18_Kemet-A_Pad1.58x1.35mm_HandSolder" H 7238 4200 50  0001 C CNN
-F 3 "~" H 7200 4350 50  0001 C CNN
-	1    7200 4350
+P 7100 4350
+F 0 "C12" H 7218 4396 50  0000 L CNN
+F 1 "4.7uf" H 7218 4305 50  0000 L CNN
+F 2 "Capacitor_Tantalum_SMD:CP_EIA-3216-18_Kemet-A_Pad1.58x1.35mm_HandSolder" H 7138 4200 50  0001 C CNN
+F 3 "~" H 7100 4350 50  0001 C CNN
+	1    7100 4350
 	1    0    0    -1
 $EndComp
@@
 	8250 4000 7550 4000
 Wire Wire Line
-	7550 4000 7200 4000
+	7550 4000 7100 4000
 Connection ~ 7550 4000
 $Comp
@@
 Text Label 6800 8450 0    50   ~ 0
 VPLL
-Text Label 6800 8950 0    50   ~ 0
-VPhy
 Wire Wire Line
 	4350 3550 4350 3400
@@
 Vcc
 Wire Wire Line
-	7200 4000 6800 4000
-Connection ~ 7200 4000
-Text Label 6900 4000 0    50   ~ 0
+	7100 4000 6800 4000
+Connection ~ 7100 4000
+Text Label 7250 4000 0    50   ~ 0
 VCore
 Wire Wire Line
@@
 F 0 "D1" H 14450 8200 50  0000 C CNN
 F 1 "LED" H 14450 8300 50  0000 C CNN
-F 2 "LED_SMD:LED_0603_1608Metric_Pad1.05x0.95mm_HandSolder" H 14300 8250 50  0001 C CNN
+F 2 "0MiscParts:LED_0603_1608Metric_Pad1.05x1.35mm_HandSolder" H 14300 8250 50  0001 C CNN
 F 3 "~" H 14300 8250 50  0001 C CNN
 	1    14300 8250
@@
 F 0 "D2" H 14450 8400 50  0000 C CNN
 F 1 "LED" H 14450 8500 50  0000 C CNN
-F 2 "LED_SMD:LED_0603_1608Metric_Pad1.05x0.95mm_HandSolder" H 14300 8450 50  0001 C CNN
+F 2 "0MiscParts:LED_0603_1608Metric_Pad1.05x1.35mm_HandSolder" H 14300 8450 50  0001 C CNN
 F 3 "~" H 14300 8450 50  0001 C CNN
 	1    14300 8450
@@
 F 0 "D3" H 14450 8600 50  0000 C CNN
 F 1 "LED" H 14450 8700 50  0000 C CNN
-F 2 "LED_SMD:LED_0603_1608Metric_Pad1.05x0.95mm_HandSolder" H 14300 8650 50  0001 C CNN
+F 2 "0MiscParts:LED_0603_1608Metric_Pad1.05x1.35mm_HandSolder" H 14300 8650 50  0001 C CNN
 F 3 "~" H 14300 8650 50  0001 C CNN
 	1    14300 8650
@@
 F 0 "D4" H 14450 8800 50  0000 C CNN
 F 1 "LED" H 14450 8900 50  0000 C CNN
-F 2 "LED_SMD:LED_0603_1608Metric_Pad1.05x0.95mm_HandSolder" H 14300 8850 50  0001 C CNN
+F 2 "0MiscParts:LED_0603_1608Metric_Pad1.05x1.35mm_HandSolder" H 14300 8850 50  0001 C CNN
 F 3 "~" H 14300 8850 50  0001 C CNN
 	1    14300 8850
@@
 F 0 "D5" H 14450 9000 50  0000 C CNN
 F 1 "LED" H 14450 9100 50  0000 C CNN
-F 2 "LED_SMD:LED_0603_1608Metric_Pad1.05x0.95mm_HandSolder" H 14300 9050 50  0001 C CNN
+F 2 "0MiscParts:LED_0603_1608Metric_Pad1.05x1.35mm_HandSolder" H 14300 9050 50  0001 C CNN
 F 3 "~" H 14300 9050 50  0001 C CNN
 	1    14300 9050
@@
 F 0 "D6" H 14450 9200 50  0000 C CNN
 F 1 "LED" H 14450 9300 50  0000 C CNN
-F 2 "LED_SMD:LED_0603_1608Metric_Pad1.05x0.95mm_HandSolder" H 14300 9250 50  0001 C CNN
+F 2 "0MiscParts:LED_0603_1608Metric_Pad1.05x1.35mm_HandSolder" H 14300 9250 50  0001 C CNN
 F 3 "~" H 14300 9250 50  0001 C CNN
 	1    14300 9250
@@
 F 0 "D7" H 14450 9400 50  0000 C CNN
 F 1 "LED" H 14450 9500 50  0000 C CNN
-F 2 "LED_SMD:LED_0603_1608Metric_Pad1.05x0.95mm_HandSolder" H 14300 9450 50  0001 C CNN
+F 2 "0MiscParts:LED_0603_1608Metric_Pad1.05x1.35mm_HandSolder" H 14300 9450 50  0001 C CNN
 F 3 "~" H 14300 9450 50  0001 C CNN
 	1    14300 9450
@@
 F 0 "D8" H 14450 9600 50  0000 C CNN
 F 1 "LED" H 14450 9700 50  0000 C CNN
-F 2 "LED_SMD:LED_0603_1608Metric_Pad1.05x0.95mm_HandSolder" H 14300 9650 50  0001 C CNN
+F 2 "0MiscParts:LED_0603_1608Metric_Pad1.05x1.35mm_HandSolder" H 14300 9650 50  0001 C CNN
 F 3 "~" H 14300 9650 50  0001 C CNN
 	1    14300 9650
@@
 	1    0    0    -1
 $EndComp
+$Comp
+L Device:R R16
+U 1 1 60631B08
+P 7650 8750
+F 0 "R16" V 7700 8500 50  0000 L CNN
+F 1 "5.1k" V 7650 8750 50  0000 C CNN
+F 2 "Resistor_SMD:R_0603_1608Metric_Pad1.05x0.95mm_HandSolder" V 7580 8750 50  0001 C CNN
+F 3 "~" H 7650 8750 50  0001 C CNN
+	1    7650 8750
+	1    0    0    -1
+$EndComp
+$Comp
+L Device:LED D9
+U 1 1 60631B0E
+P 7650 9450
+F 0 "D9" H 7800 9400 50  0000 C CNN
+F 1 "LED" H 7800 9500 50  0000 C CNN
+F 2 "0MiscParts:LED_0603_1608Metric_Pad1.05x1.35mm_HandSolder" H 7650 9450 50  0001 C CNN
+F 3 "~" H 7650 9450 50  0001 C CNN
+	1    7650 9450
+	0    -1   -1   0
+$EndComp
+$Comp
+L power:GND #PWR0101
+U 1 1 60631B15
+P 7650 9600
+F 0 "#PWR0101" H 7650 9350 50  0001 C CNN
+F 1 "GND" H 7655 9427 50  0000 C CNN
+F 2 "" H 7650 9600 50  0001 C CNN
+F 3 "" H 7650 9600 50  0001 C CNN
+	1    7650 9600
+	1    0    0    -1
+$EndComp
+Wire Wire Line
+	7650 8900 7650 9300
+Text Label 6800 8950 0    50   ~ 0
+VPhy
+Wire Wire Line
+	6050 8950 7000 8950
+$Comp
+L power:+3.3V #PWR0102
+U 1 1 6064EE2F
+P 7650 8600
+F 0 "#PWR0102" H 7650 8450 50  0001 C CNN
+F 1 "+3.3V" H 7665 8773 50  0000 C CNN
+F 2 "" H 7650 8600 50  0001 C CNN
+F 3 "" H 7650 8600 50  0001 C CNN
+	1    7650 8600
+	1    0    0    -1
+$EndComp
+Text Label 7650 9100 0    50   ~ 0
+3.3VR
 $EndSCHEMATC

Commit message: Updating component values.  Updates for new Kicad version.
Parts:
- CR1, CR2: symbol 00User:ProtectionDiode -> FT4232-rescue:ProtectionDiode-00User
- J1: symbol Connector:USB_B_Mini -> FT4232-rescue:USB_B_Mini-Connector
Changed lines of the file:
@@
 	6500 4750 6150 4750
 $Comp
-L 00User:ProtectionDiode CR2
+L FT4232-rescue:ProtectionDiode-00User CR2
 U 1 1 6009C527
 P 5600 5350
@@
 $EndComp
 $Comp
-L 00User:ProtectionDiode CR1
+L FT4232-rescue:ProtectionDiode-00User CR1
 U 1 1 6009D10D
 P 5200 5350
@@
 $EndComp
 $Comp
-L Connector:USB_B_Mini J1
+L FT4232-rescue:USB_B_Mini-Connector J1
 U 1 1 600A20BC
 P 4050 4850

Commit message: Updates to component values.
Parts:
- D1, D3, D5, D7, D9: value LED -> LED Gr
- D2, D4, D6, D8: value LED -> LED Yl
- R10, R12, R14, R16, R8: value 5.1k -> 2.4k
- R11, R13, R15, R9: value 5.1k -> 1k
Changed lines of the file:
@@
 P 13600 8250
 F 0 "R8" V 13650 8000 50  0000 L CNN
-F 1 "5.1k" V 13600 8250 50  0000 C CNN
+F 1 "2.4k" V 13600 8250 50  0000 C CNN
 F 2 "Resistor_SMD:R_0603_1608Metric_Pad1.05x0.95mm_HandSolder" V 13530 8250 50  0001 C CNN
 F 3 "~" H 13600 8250 50  0001 C CNN
@@
 P 14300 8250
 F 0 "D1" H 14450 8200 50  0000 C CNN
-F 1 "LED" H 14450 8300 50  0000 C CNN
+F 1 "LED Gr" H 14500 8300 50  0000 C CNN
 F 2 "0MiscParts:LED_0603_1608Metric_Pad1.05x1.35mm_HandSolder" H 14300 8250 50  0001 C CNN
 F 3 "~" H 14300 8250 50  0001 C CNN
@@
 P 13600 8450
 F 0 "R9" V 13650 8200 50  0000 L CNN
-F 1 "5.1k" V 13600 8450 50  0000 C CNN
+F 1 "1k" V 13600 8450 50  0000 C CNN
 F 2 "Resistor_SMD:R_0603_1608Metric_Pad1.05x0.95mm_HandSolder" V 13530 8450 50  0001 C CNN
 F 3 "~" H 13600 8450 50  0001 C CNN
@@
 P 14300 8450
 F 0 "D2" H 14450 8400 50  0000 C CNN
-F 1 "LED" H 14450 8500 50  0000 C CNN
+F 1 "LED Yl" H 14500 8500 50  0000 C CNN
 F 2 "0MiscParts:LED_0603_1608Metric_Pad1.05x1.35mm_HandSolder" H 14300 8450 50  0001 C CNN
 F 3 "~" H 14300 8450 50  0001 C CNN
@@
 P 13600 8650
 F 0 "R10" V 13650 8400 50  0000 L CNN
-F 1 "5.1k" V 13600 8650 50  0000 C CNN
+F 1 "2.4k" V 13600 8650 50  0000 C CNN
 F 2 "Resistor_SMD:R_0603_1608Metric_Pad1.05x0.95mm_HandSolder" V 13530 8650 50  0001 C CNN
 F 3 "~" H 13600 8650 50  0001 C CNN
@@
 P 14300 8650
 F 0 "D3" H 14450 8600 50  0000 C CNN
-F 1 "LED" H 14450 8700 50  0000 C CNN
+F 1 "LED Gr" H 14500 8700 50  0000 C CNN
 F 2 "0MiscParts:LED_0603_1608Metric_Pad1.05x1.35mm_HandSolder" H 14300 8650 50  0001 C CNN
 F 3 "~" H 14300 8650 50  0001 C CNN
@@
 P 13600 8850
 F 0 "R11" V 13650 8600 50  0000 L CNN
-F 1 "5.1k" V 13600 8850 50  0000 C CNN
+F 1 "1k" V 13600 8850 50  0000 C CNN
 F 2 "Resistor_SMD:R_0603_1608Metric_Pad1.05x0.95mm_HandSolder" V 13530 8850 50  0001 C CNN
 F 3 "~" H 13600 8850 50  0001 C CNN
@@
 P 14300 8850
 F 0 "D4" H 14450 8800 50  0000 C CNN
-F 1 "LED" H 14450 8900 50  0000 C CNN
+F 1 "LED Yl" H 14500 8900 50  0000 C CNN
 F 2 "0MiscParts:LED_0603_1608Metric_Pad1.05x1.35mm_HandSolder" H 14300 8850 50  0001 C CNN
 F 3 "~" H 14300 8850 50  0001 C CNN
@@
 P 13600 9050
 F 0 "R12" V 13650 8800 50  0000 L CNN
-F 1 "5.1k" V 13600 9050 50  0000 C CNN
+F 1 "2.4k" V 13600 9050 50  0000 C CNN
 F 2 "Resistor_SMD:R_0603_1608Metric_Pad1.05x0.95mm_HandSolder" V 13530 9050 50  0001 C CNN
 F 3 "~" H 13600 9050 50  0001 C CNN
@@
 P 14300 9050
 F 0 "D5" H 14450 9000 50  0000 C CNN
-F 1 "LED" H 14450 9100 50  0000 C CNN
+F 1 "LED Gr" H 14500 9100 50  0000 C CNN
 F 2 "0MiscParts:LED_0603_1608Metric_Pad1.05x1.35mm_HandSolder" H 14300 9050 50  0001 C CNN
 F 3 "~" H 14300 9050 50  0001 C CNN
@@
 P 13600 9250
 F 0 "R13" V 13650 9000 50  0000 L CNN
-F 1 "5.1k" V 13600 9250 50  0000 C CNN
+F 1 "1k" V 13600 9250 50  0000 C CNN
 F 2 "Resistor_SMD:R_0603_1608Metric_Pad1.05x0.95mm_HandSolder" V 13530 9250 50  0001 C CNN
 F 3 "~" H 13600 9250 50  0001 C CNN
@@
 P 14300 9250
 F 0 "D6" H 14450 9200 50  0000 C CNN
-F 1 "LED" H 14450 9300 50  0000 C CNN
+F 1 "LED Yl" H 14500 9300 50  0000 C CNN
 F 2 "0MiscParts:LED_0603_1608Metric_Pad1.05x1.35mm_HandSolder" H 14300 9250 50  0001 C CNN
 F 3 "~" H 14300 9250 50  0001 C CNN
@@
 P 13600 9450
 F 0 "R14" V 13650 9200 50  0000 L CNN
-F 1 "5.1k" V 13600 9450 50  0000 C CNN
+F 1 "2.4k" V 13600 9450 50  0000 C CNN
 F 2 "Resistor_SMD:R_0603_1608Metric_Pad1.05x0.95mm_HandSolder" V 13530 9450 50  0001 C CNN
 F 3 "~" H 13600 9450 50  0001 C CNN
@@
 P 14300 9450
 F 0 "D7" H 14450 9400 50  0000 C CNN
-F 1 "LED" H 14450 9500 50  0000 C CNN
+F 1 "LED Gr" H 14500 9500 50  0000 C CNN
 F 2 "0MiscParts:LED_0603_1608Metric_Pad1.05x1.35mm_HandSolder" H 14300 9450 50  0001 C CNN
 F 3 "~" H 14300 9450 50  0001 C CNN
@@
 P 13600 9650
 F 0 "R15" V 13650 9400 50  0000 L CNN
-F 1 "5.1k" V 13600 9650 50  0000 C CNN
+F 1 "1k" V 13600 9650 50  0000 C CNN
 F 2 "Resistor_SMD:R_0603_1608Metric_Pad1.05x0.95mm_HandSolder" V 13530 9650 50  0001 C CNN
 F 3 "~" H 13600 9650 50  0001 C CNN
@@
 P 14300 9650
 F 0 "D8" H 14450 9600 50  0000 C CNN
-F 1 "LED" H 14450 9700 50  0000 C CNN
+F 1 "LED Yl" H 14500 9700 50  0000 C CNN
 F 2 "0MiscParts:LED_0603_1608Metric_Pad1.05x1.35mm_HandSolder" H 14300 9650 50  0001 C CNN
 F 3 "~" H 14300 9650 50  0001 C CNN
@@
 P 7650 8750
 F 0 "R16" V 7700 8500 50  0000 L CNN
-F 1 "5.1k" V 7650 8750 50  0000 C CNN
+F 1 "2.4k" V 7650 8750 50  0000 C CNN
 F 2 "Resistor_SMD:R_0603_1608Metric_Pad1.05x0.95mm_HandSolder" V 7580 8750 50  0001 C CNN
 F 3 "~" H 7650 8750 50  0001 C CNN
@@
 P 7650 9450
 F 0 "D9" H 7800 9400 50  0000 C CNN
-F 1 "LED" H 7800 9500 50  0000 C CNN
+F 1 "LED Gr" H 7650 9550 50  0000 C CNN
 F 2 "0MiscParts:LED_0603_1608Metric_Pad1.05x1.35mm_HandSolder" H 7650 9450 50  0001 C CNN
 F 3 "~" H 7650 9450 50  0001 C CNN
