File: STM32F1/STM32F1.sch (KiCad schematic (older format))
At the start: 40 parts, among them J1 Conn_02x03_Odd_Even, J2 Conn_01x04_Male, J3 10033526-N3212MLF, J4 Conn_01x20_Male, J5 Conn_01x20_Male, SW1 PTS 647 SK38 SMTR2 LFS, U1 RT9193, U2 STM32F103CBTx, Y1 ABL-8.000MHZ-B2‎, Y2 RSM200S-32.768-12.5-10PPM-NPB

Commit message: Update LED resistor values.
Parts:
- R10: value 10k -> 2.4k
- R11: value 10k -> 1k
Changed lines of the file:
@@
 P 9350 1550
 F 0 "R10" H 9420 1596 50  0000 L CNN
-F 1 "10k" H 9420 1505 50  0000 L CNN
+F 1 "2.4k" H 9420 1505 50  0000 L CNN
 F 2 "Resistor_SMD:R_0603_1608Metric_Pad1.05x0.95mm_HandSolder" V 9280 1550 50  0001 C CNN
 F 3 "~" H 9350 1550 50  0001 C CNN
@@
 P 9800 1550
 F 0 "R11" H 9870 1596 50  0000 L CNN
-F 1 "10k" H 9870 1505 50  0000 L CNN
+F 1 "1k" H 9870 1505 50  0000 L CNN
 F 2 "Resistor_SMD:R_0603_1608Metric_Pad1.05x0.95mm_HandSolder" V 9730 1550 50  0001 C CNN
 F 3 "~" H 9800 1550 50  0001 C CNN

Commit message: Updating component values.  Updates for new Kicad version.
Parts:
- J3: symbol Connector:USB_B_Mini -> STM32F1-rescue:USB_B_Mini-Connector
Changed lines of the file:
@@
 $EndComp
 $Comp
-L Connector:USB_B_Mini J3
+L STM32F1-rescue:USB_B_Mini-Connector J3
 U 1 1 5EF8B8E4
 P 7350 1800

Commit message: Updates to component values.
Parts:
- U1: symbol 00User:RT9193 -> STM32F1-rescue:RT9193-00User
- Y2: symbol 00User:Crystal_4_Pads -> STM32F1-rescue:Crystal_4_Pads-00User
Changed lines of the file:
@@
 	2150 3700 2150 3850
 $Comp
-L 00User:Crystal_4_Pads Y2
+L STM32F1-rescue:Crystal_4_Pads-00User Y2
 U 1 1 5F086BCB
 P 1150 4350
@@
 $EndComp
 $Comp
-L 00User:RT9193 U1
+L STM32F1-rescue:RT9193-00User U1
 U 1 1 5EF70C32
 P 2150 6750
