File: STM32F1/STM32F1.sch (KiCad schematic (older format))
At the start: 40 parts, among them J1 Conn_02x03_Odd_Even, J2 Conn_01x04_Male, J3 10033526-N3212MLF, J4 Conn_01x20_Male, J5 Conn_01x20_Male, SW1 PTS 647 SK38 SMTR2 LFS, U1 RT9193, U2 STM32F103CBTx, Y1 ABL-8.000MHZ-B2‎, Y2 RSM200S-32.768-12.5-10PPM-NPB

Commit message: STM32F1 board with different crystals.
Parts:
- removed R2: R, Resistor_SMD:R_0603_1608Metric_Pad1.05x0.95mm_HandSolder, symbol Device:R
- removed Y1: ABL-8.000MHZ-B2‎, Crystal:Crystal_HC49-4H_Vertical, symbol Device:Crystal
- removed Y2: RSM200S-32.768-12.5-10PPM-NPB, 0MiscParts:RSM2000S, symbol 00User:Crystal_4_Pads
- added Y1: ABM3BAIG-8.000MHZ-1Z-T, SamacSys_Parts:ABM3BAIG8000MHZ1ZT, symbol SamacSys_Parts:ABM3BAIG-8.000MHZ-1Z-T
- added Y2: CM7V-T1A-32.768k-9pF-20PPM-TA-QA_T3, SamacSys_Parts:CM7VT1A32768kHz125pF10PPMTBQC, symbol SamacSys_Parts:CM7V-T1A-32.768k-9pF-20PPM-TA-QA_T3
- D3, D4: footprint LED_SMD:LED_0603_1608Metric_Pad1.05x0.95mm_HandSolder -> 0MiscParts:LED_0603_1608Metric_Pad1.05x1.35mm_HandSolder
Connections:
- wire segments 158 -> 160
Changed lines of the file:
@@
-$EndComp
-$Comp
-L Device:Crystal Y1
-U 1 1 5EF634D1
-P 1150 3250
-F 0 "Y1" H 1150 3518 50  0000 C CNN
-F 1 "ABL-8.000MHZ-B2‎ " H 1150 3427 50  0000 C CNN
-F 2 "Crystal:Crystal_HC49-4H_Vertical" H 1150 3250 50  0001 C CNN
-F 3 "~" H 1150 3250 50  0001 C CNN
-	1    1150 3250
-	1    0    0    -1
 $EndComp
 $Comp
@@
 	2150 3700 2150 3850
 $Comp
-L 00User:Crystal_4_Pads Y2
-U 1 1 5F086BCB
-P 1150 4350
-F 0 "Y2" H 1150 4618 50  0000 C CNN
-F 1 "RSM200S-32.768-12.5-10PPM-NPB" H 1150 4527 50  0000 C CNN
-F 2 "0MiscParts:RSM2000S" H 1150 4350 50  0001 C CNN
-F 3 "~" H 1150 4350 50  0001 C CNN
-	1    1150 4350
-	1    0    0    -1
-$EndComp
-$Comp
 L power:+3.3V #PWR034
 U 1 1 5F0CFE2C
@@
 $EndComp
 $Comp
-L Device:R R2
-U 1 1 5F0E4BE6
-P 1150 2900
-F 0 "R2" V 943 2900 50  0000 C CNN
-F 1 "R" V 1034 2900 50  0000 C CNN
-F 2 "Resistor_SMD:R_0603_1608Metric_Pad1.05x0.95mm_HandSolder" V 1080 2900 50  0001 C CNN
-F 3 "~" H 1150 2900 50  0001 C CNN
-	1    1150 2900
-	0    1    1    0
-$EndComp
-Wire Wire Line
-	1000 2900 650  2900
-Wire Wire Line
-	1300 2900 1650 2900
-Text Label 700  2900 0    50   ~ 0
-D0
-Text Label 1500 2900 0    50   ~ 0
-D1
-$Comp
 L power:+3.3V #PWR043
 U 1 1 5F10EB21
@@
 F 0 "D3" V 9389 1033 50  0000 R CNN
 F 1 "LED" V 9298 1033 50  0000 R CNN
-F 2 "LED_SMD:LED_0603_1608Metric_Pad1.05x0.95mm_HandSolder" H 9350 1150 50  0001 C CNN
+F 2 "0MiscParts:LED_0603_1608Metric_Pad1.05x1.35mm_HandSolder" H 9350 1150 50  0001 C CNN
 F 3 "~" H 9350 1150 50  0001 C CNN
 	1    9350 1150
@@
 F 0 "D4" V 9839 1033 50  0000 R CNN
 F 1 "LED" V 9748 1033 50  0000 R CNN
-F 2 "LED_SMD:LED_0603_1608Metric_Pad1.05x0.95mm_HandSolder" H 9800 1150 50  0001 C CNN
+F 2 "0MiscParts:LED_0603_1608Metric_Pad1.05x1.35mm_HandSolder" H 9800 1150 50  0001 C CNN
 F 3 "~" H 9800 1150 50  0001 C CNN
 	1    9800 1150
@@
 Text Label 9300 3850 0    50   ~ 0
 5VIn
+$Comp
+L SamacSys_Parts:ABM3BAIG-8.000MHZ-1Z-T Y1
+U 1 1 60398552
+P -2700 3400
+F 0 "Y1" H -1900 3665 50  0000 C CNN
+F 1 "ABM3BAIG-8.000MHZ-1Z-T" H -1900 3574 50  0000 C CNN
+F 2 "SamacSys_Parts:ABM3BAIG8000MHZ1ZT" H -1250 3500 50  0001 L CNN
+F 3 "https://componentsearchengine.com/Datasheets/1/ABM3BAIG-8.000MHZ-1Z-T.pdf" H -1250 3400 50  0001 L CNN
+F 4 "Crystals 18pF 8MHz 10ppm AEC-Q200 -40C +125C" H -1250 3300 50  0001 L CNN "Description"
+F 5 "0.9" H -1250 3200 50  0001 L CNN "Height"
+F 6 "815-M3BAIG-8-1ZT" H -1250 3100 50  0001 L CNN "Mouser Part Number"
+F 7 "https://www.mouser.co.uk/ProductDetail/ABRACON/ABM3BAIG-8000MHZ-1Z-T/?qs=uwxL4vQweFMtl1NAFNP1Qg%3D%3D" H -1250 3000 50  0001 L CNN "Mouser Price/Stock"
+F 8 "ABRACON" H -1250 2900 50  0001 L CNN "Manufacturer_Name"
+F 9 "ABM3BAIG-8.000MHZ-1Z-T" H -1250 2800 50  0001 L CNN "Manufacturer_Part_Number"
+	1    -2700 3400
+	1    0    0    -1
+$EndComp
+$Comp
+L SamacSys_Parts:CM7V-T1A-32.768k-9pF-20PPM-TA-QA_T3 Y2
+U 1 1 60399300
+P -2350 4550
+F 0 "Y2" H -1722 4546 50  0000 L CNN
+F 1 "CM7V-T1A-32.768k-9pF-20PPM-TA-QA_T3" H -1722 4455 50  0000 L CNN
+F 2 "SamacSys_Parts:CM7VT1A32768kHz125pF10PPMTBQC" H -1700 4650 50  0001 L CNN
+F 3 "https://componentsearchengine.com/Datasheets/1/CM7V-T1A-32.768k-9pF-20PPM-TA-QA T3.pdf" H -1700 4550 50  0001 L CNN
+F 4 "Crystals 32.768 kHz 9.0 pF +/-20 PPM AEC-Q200" H -1700 4450 50  0001 L CNN "Description"
+F 5 "0.65" H -1700 4350 50  0001 L CNN "Height"
+F 6 "428-201568-MG03" H -1700 4250 50  0001 L CNN "Mouser Part Number"
+F 7 "https://www.mouser.co.uk/ProductDetail/Micro-Crystal/CM7V-T1A-32768k-9pF-20PPM-TA-QA-T3?qs=chTDxNqvsykvxHA%2FArNuyw%3D%3D" H -1700 4150 50  0001 L CNN "Mouser Price/Stock"
+F 8 "Micro Crystal AG" H -1700 4050 50  0001 L CNN "Manufacturer_Name"
+F 9 "CM7V-T1A-32.768k-9pF-20PPM-TA-QA T3" H -1700 3950 50  0001 L CNN "Manufacturer_Part_Number"
+	1    -2350 4550
+	1    0    0    -1
+$EndComp
+Wire Wire Line
+	-2700 3500 -3050 3500
+Text Label -3000 3500 0    50   ~ 0
+D0
+Wire Wire Line
+	-850 3400 -1100 3400
+Text Label -1000 3400 0    50   ~ 0
+D1
+Wire Wire Line
+	-2350 4550 -2600 4550
+Text Label -2550 4550 0    50   ~ 0
+C14
+Wire Wire Line
+	-2350 4650 -2600 4650
+Text Label -2550 4650 0    50   ~ 0
+C15
+$Comp
+L power:GND #PWR?
+U 1 1 60475233
+P -1100 3500
+F 0 "#PWR?" H -1100 3250 50  0001 C CNN
+F 1 "GND" V -1100 3300 50  0000 C CNN
+F 2 "" H -1100 3500 50  0001 C CNN
+F 3 "" H -1100 3500 50  0001 C CNN
+	1    -1100 3500
+	0    -1   -1   0
+$EndComp
+$Comp
+L power:GND #PWR?
+U 1 1 60475B72
+P -2700 3400
+F 0 "#PWR?" H -2700 3150 50  0001 C CNN
+F 1 "GND" V -2750 3200 50  0000 C CNN
+F 2 "" H -2700 3400 50  0001 C CNN
+F 3 "" H -2700 3400 50  0001 C CNN
+	1    -2700 3400
+	0    1    1    0
+$EndComp
 $EndSCHEMATC

Commit message: STM32F1 new layout.
Parts:
- removed J1: Conn_02x03_Odd_Even, Connector_PinHeader_2.54mm:PinHeader_2x03_P2.54mm_Vertical, symbol Connector_Generic:Conn_02x03_Odd_Even
- removed Y2: CM7V-T1A-32.768k-9pF-20PPM-TA-QA_T3, SamacSys_Parts:CM7VT1A32768kHz125pF10PPMTBQC, symbol SamacSys_Parts:CM7V-T1A-32.768k-9pF-20PPM-TA-QA_T3
- added JP1, JP2: Jumper_3_Open, 0MiscParts:Jumper_0603_3, symbol Jumper:Jumper_3_Open
- added JP3, JP4, JP5: Jumper_NO_Small, Resistor_SMD:R_0603_1608Metric_Pad0.98x0.95mm_HandSolder, symbol Device:Jumper_NO_Small
- added Y2: Crystal_GND2_Small, 0MiscParts:Crystal_ECX-34G, symbol Device:Crystal_GND2_Small
- U1: symbol 00User:RT9193 -> STM32F1-rescue:RT9193-00User
- Y1: footprint SamacSys_Parts:ABM3BAIG8000MHZ1ZT -> 0MiscParts:Crystal_ABM3BAIG_5x3.2; symbol SamacSys_Parts:ABM3BAIG-8.000MHZ-1Z-T -> STM32F1-rescue:ABM3BAIG-8.000MHZ-1Z-T-SamacSys_Parts
- renumbered C7 to C5, C8 to C7, C5 to C8, J2 to J1, J3 to J2, J4 to J3, J5 to J4, R4 to R2, R5 to R3, R6 to R4, R7 to R5, R8 to R6, R9 to R7, R10 to R8, R11 to R9
Connections:
- net labels added: C14Ext, C15Ext
- wire segments 160 -> 161
Other:
- moved on the sheet: C2, C3, C5, C6, C8, R1, R2, SW1, Y1
