File: STM32F1MonA/STM32F1MonA.kicad_pcb (KiCad board)
At the start: 2 copper layers, 55.2 x 41.3 mm, 37 parts, among them J1 PJ-102, J2 Conn_01x03_Female, J3 RJ45, J4 Conn_01x02, J5 Conn_01x03_Male, J6 RJ45, J7 Conn_01x20_Male, J8 Conn_02x04_Odd_Even, J9 Conn_02x04_Odd_Even, U1 AP1117-50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

Commit message: Updates while making boards.
Other:
- board text added: "G"
- board text added: "Rx"
- board text added: "Tx"
